File: ShinyBoost/ShinyBoost.kicad_sch (KiCad schematic)
At the start: 26 parts

Commit message: Work on sims
Parts:
- removed C? (x3): 1uF, symbol Device:C
- removed C? (x2): 330uF, symbol Device:CP1
- removed C?: C, symbol Device:C
- removed D?: D_Schottky, symbol Device:D_Schottky
- removed L?: 1mH, symbol Device:L
- removed Q?: Q_NMOS_GDS, symbol Device:Q_NMOS_GDS
- removed R? (x4): 10K, symbol Device:R_US
- removed R?: 2.5K, symbol Device:R_US
- removed R?: 1.7K, symbol Device:R_US
- removed R? (x2): 47K, symbol Device:R_US
- removed R?: 100K, symbol Device:R_US
- removed RV?: 10K, symbol Device:R_POT_US
- removed U? (x5): MCP6004, symbol Amplifier_Operational:MCP6004
- removed U?: ATmega328PB-MU, Package_DFN_QFN:QFN-32-1EP_5x5mm_P0.5mm_EP3.1x3.1mm, symbol MCU_Microchip_ATmega:ATmega328PB-MU
Other:
- moved on the sheet: J?
